File: stacja_mierzaca/stacja_mierzaca.kicad_sch (KiCad schematic)
At the start: 14 parts, among them M1 HW373-TP4056, Q1 PMOS, U1 ESP32-WROOM32-DEVKIT-V1-30P, U2 SOIL_DS18B20, U3 Ai-Thinker-Ra-02

Commit message: feat(end_device): updated end device schematic to include SX1276 module
Parts:
- removed U3: Ai-Thinker-Ra-02, RF_Module:Ai-Thinker-Ra-01-LoRa, symbol RF_Module:Ai-Thinker-Ra-02
- added U4: (no value), symbol Custom_RF_Modules:SX1276_Module
- VR1: value ~ -> (none)
Connections:
- net VDD_3V3: no longer U1.16 (3V3)
- net RA02_DIO0 renamed SX1276_DIO0
- net SX1276_DIO0: now also U4.14 (DIO0)
- net RA02_DIO1 renamed SX1276_DIO1
- net SX1276_DIO1: now also U4.15 (DIO1)
- net RA02_MISO renamed SX1276_MISO
- net SX1276_MISO: now also U4.7 (MISO)
- net RA02_MOSI renamed SX1276_MOSI
- net SX1276_MOSI: now also U4.6 (MOSI)
- net RA02_RESET renamed SX1276_REST
- net SX1276_REST: now also U4.3 (REST)
- net RA02_SCK renamed SX1276_SCK
- net SX1276_SCK: now also U4.5 (SCK)
- net RA02_SS renamed SX1276_SS
- net SX1276_SS: now also U4.4 (NSS)
- new net VCC_3V3: U1.16 (3V3), U4.13 (VCC)
